Commit message: urdf basic

File: src/dd_bot/description/gazebo_control.xacro (robot description, xacro)
@@ -6,5 +6,5 @@
             <left_joint>left_wheel_joint</left_joint>
             <right_joint>right_wheel_joint</right_joint>
-            <wheel_separation>0.54</wheel_separation>
+            <wheel_separation>0.56</wheel_separation>
             <wheel_radius>0.1</wheel_radius>
             <!-- Limits -->

File: src/dd_bot/description/robot_core.xacro (robot description, xacro)
@@ -63,7 +63,10 @@
             </geometry>
         </collision>
-        <xacro:inertial_box mass="0.5" x="0.75" y="0.5" z="0.03" >
-            <origin xyz="0 0.0 0.0" rpy="0 0 0"/>
-        </xacro:inertial_box>
+        <inertial>
+        <origin xyz="0.20 0.0 0" rpy="0 0 0"/>
+        <mass value="1.9809343e+01"/>
+        <inertia ixx="4.914e-01" iyy="2.317e-01" izz="5.354e-01"
+                ixy="3.367e-16" ixz="-7.465e-03" iyz="1.793e-16"/>
+        </inertial>
     </link>
     <gazebo reference="chassis">
